Commit message: add cov estimation, still working

File: src/stair_mapping/urdf/hex_mini_model.urdf (robot description, URDF)
Before this commit: robot hex_mini, 7 links, 6 joints
Joints:
- joint joint_camera_to_base: origin xyz=0.22 0 0.26 rpy=0 2.02 -0.04 -> xyz=0.22 0 0.26 rpy=0 2.05 -0.04

Commit message: add laser match's infomation matrix to pose graph

File: src/stair_mapping/urdf/hex_mini_model.urdf (robot description, URDF)
Before this commit: robot hex_mini, 7 links, 6 joints
Joints:
- joint joint_camera_to_base: origin xyz=0.22 0 0.26 rpy=0 2.05 -0.04 -> xyz=0.22 0 0.26 rpy=0 2.09 -0.04

Commit message: tunning

File: src/stair_mapping/urdf/hex_mini_model.urdf (robot description, URDF)
Before this commit: robot hex_mini, 7 links, 6 joints
Joints:
- joint joint_camera_to_base: origin xyz=0.22 0 0.26 rpy=0 2.09 -0.04 -> xyz=0.22 0 0.26 rpy=0 2.05 -0.04

Commit message: tunning, small imu correction is adequate

File: src/stair_mapping/urdf/hex_mini_model.urdf (robot description, URDF)
Before this commit: robot hex_mini, 7 links, 6 joints
Joints:
- joint joint_camera_to_base: origin xyz=0.22 0 0.26 rpy=0 2.05 -0.04 -> xyz=0.22 0 0.26 rpy=0 2.06 0.0

Commit message: add foothold check

File: src/stair_mapping/urdf/hex_mini_model.urdf (robot description, URDF)
Before this commit: robot hex_mini, 7 links, 6 joints
Links:
- link body_link: geometry collision box size=0.5 0.3 0.1; visual box size=0.68 0.35 0.13
Joints:
- joint joint_camera_to_base: origin xyz=0.22 0 0.26 rpy=0 2.06 0.0 -> xyz=0.20 0 0.26 rpy=0 2.06 0.0

Commit message: add ground true for calibration

File: src/stair_mapping/urdf/hex_mini_model.urdf (robot description, URDF)
Before this commit: robot hex_mini, 7 links, 6 joints
Joints:
- joint joint_camera_to_base: origin xyz=0.20 0 0.26 rpy=0 2.06 0.0 -> xyz=0.19 0 0.28 rpy=0 2.06 -0.04

Commit message: add Z drift compensation (naive aproach)

File: src/stair_mapping/urdf/hex_mini_model.urdf (robot description, URDF)
Before this commit: robot hex_mini, 7 links, 6 joints
Joints:
- joint joint_camera_to_base: origin xyz=0.19 0 0.28 rpy=0 2.06 -0.04 -> xyz=0.19 0 0.265 rpy=0 2.06 -0.04

Commit message: tuning

File: src/stair_mapping/urdf/hex_mini_model.urdf (robot description, URDF)
Before this commit: robot hex_mini, 7 links, 6 joints
Joints:
- joint joint_camera_to_base: origin xyz=0.19 0 0.265 rpy=0 2.06 -0.04 -> xyz=0.19 0 0.265 rpy=-0.06 2.08 -0.08

Commit message: adopt to all message version

File: src/stair_mapping/urdf/hex_mini_model.urdf (robot description, URDF)
Before this commit: robot hex_mini, 7 links, 6 joints
Joints:
- joint joint_camera_to_base: origin xyz=0.19 0 0.265 rpy=-0.06 2.08 -0.08 -> xyz=0.19 0 0.265 rpy=-0.06 2.09 -0.08

Commit message: ongoing

File: src/stair_mapping/urdf/hex_mini_model.urdf (robot description, URDF)
Before this commit: robot hex_mini, 7 links, 6 joints
Joints:
- joint joint_camera_to_base: origin xyz=0.19 0 0.265 rpy=-0.06 2.09 -0.08 -> xyz=0.22 0 0.26 rpy=0 2.05 -0.04

Commit message: Ready to use RGBD odometry

File: src/stair_mapping/urdf/hex_mini_model.urdf (robot description, URDF)
Before this commit: robot hex_mini, 7 links, 6 joints
Joints:
- joint joint_camera_to_base: origin xyz=0.22 0 0.26 rpy=0 2.05 -0.04 -> xyz=0.19 0 0.265 rpy=-0.06 2.09 -0.08

Commit message: recalibrated

File: src/stair_mapping/urdf/hex_mini_model.urdf (robot description, URDF)
Before this commit: robot hex_mini, 7 links, 6 joints
Joints:
- joint joint_camera_to_base: origin xyz=0.22 0 0.26 rpy=0 2.05 -0.04 -> xyz=0.28 0 0.25 rpy=-0.05 2.19 0.0

Commit message: calibrated

File: src/stair_mapping/urdf/hex_mini_model.urdf (robot description, URDF)
Before this commit: robot hex_mini, 7 links, 6 joints
Joints:
- joint joint_camera_to_base: origin xyz=0.28 0 0.25 rpy=-0.05 2.19 0.0 -> xyz=0.30 0 0.25 rpy=-0.05 2.19 0.0

Commit message: add rgbd odometry ok

File: src/stair_mapping/urdf/hex_mini_model.urdf (robot description, URDF)
Before this commit: robot hex_mini, 7 links, 6 joints
Joints:
- joint joint_camera_to_base: origin xyz=0.30 0 0.25 rpy=-0.05 2.19 0.0 -> xyz=0.32 0 0.29 rpy=-0.05 2.19 0.0

Commit message: try solving mismatch plane prob

File: src/stair_mapping/urdf/hex_mini_model.urdf (robot description, URDF)
Before this commit: robot hex_mini, 7 links, 6 joints
Joints:
- joint joint_camera_to_base: origin xyz=0.30 0 0.25 rpy=-0.05 2.19 0.0 -> xyz=0.27 0 0.25 rpy=-0.05 2.19 0.0

Commit message: fix bug: use info matrix that is square-rooted may cause strange large drift, use info matrix not square-rooted is ok otherwise

File: src/stair_mapping/urdf/hex_mini_model.urdf (robot description, URDF)
Before this commit: robot hex_mini, 7 links, 6 joints
Joints:
- joint joint_camera_to_base: origin xyz=0.27 0 0.25 rpy=-0.05 2.19 0.0 -> xyz=0.27 0 0.25 rpy=0.03 2.22 0.03

Commit message: fix infomatrix bug and f2f odom transform bug

File: src/stair_mapping/urdf/hex_mini_model.urdf (robot description, URDF)
Before this commit: robot hex_mini, 7 links, 6 joints
Joints:
- joint joint_camera_to_base: origin xyz=0.19 0 0.265 rpy=-0.06 2.08 -0.08 -> xyz=0.27 0 0.265 rpy=0.03 2.20 0.03

Commit message: Refracting: Match pcls with camera local frame

File: src/stair_mapping/urdf/hex_mini_model.urdf (robot description, URDF)
Before this commit: robot hex_mini, 7 links, 6 joints
Joints:
- joint joint_camera_to_base: origin xyz=0.27 0 0.265 rpy=0.03 2.20 0.03 -> xyz=0.27 0 0.25 rpy=0.03 2.22 0.03
